Commit message: ...

File: src/pipe_bringup/urdf/pipe_bot.urdf.xacro (robot description, xacro)
@@ -1,10 +1,9 @@
 <?xml version="1.0"?>
 <robot xmlns:xacro="http://www.ros.org/wiki/xacro" name="pipe_bot">
-  <!-- Base link -->
+  <link name="base_footprint"/>
   <link name="base_link">
     <visual>
-      <origin xyz="0 0 0" rpy="0 0 0"/>
-      <geometry>
-        <box size="0.3 0.2 0.1"/>
+      <geometry>
+        <box size="0.30 0.18 0.08"/>
       </geometry>
       <material name="blue">
@@ -13,200 +12,161 @@
     </visual>
     <collision>
-      <origin xyz="0 0 0" rpy="0 0 0"/>
-      <geometry>
-        <box size="0.3 0.2 0.1"/>
-      </geometry>
-    </collision>
-    <inertial>
-      <origin xyz="0 0 0" rpy="0 0 0"/>
-      <mass value="2.0"/>
-      <inertia ixx="0.01" ixy="0.0" ixz="0.0" iyy="0.01" iyz="0.0" izz="0.01"/>
-    </inertial>
-  </link>
-  <!-- Gazebo material for base_link -->
+      <geometry>
+        <box size="0.30 0.18 0.08"/>
+      </geometry>
+    </collision>
+    <inertial>
+      <mass value="8.0"/>
+      <inertia ixx="0.02" ixy="0" ixz="0" iyy="0.03" iyz="0" izz="0.04"/>
+    </inertial>
+  </link>
+  <joint name="base_joint" type="fixed">
+    <parent link="base_footprint"/>
+    <child link="base_link"/>
+    <origin xyz="0 0 0.06" rpy="0 0 0"/>
+  </joint>
   <gazebo reference="base_link">
     <material>Gazebo/Blue</material>
   </gazebo>
-  <!-- Front Left Wheel -->
   <link name="wheel_fl">
     <visual>
       <origin xyz="0 0 0" rpy="1.5708 0 0"/>
       <geometry>
-        <cylinder radius="0.03" length="0.02"/>
-      </geometry>
-      <material name="black">
-        <color rgba="0 0 0 1"/>
-      </material>
-    </visual>
-    <collision>
-      <origin xyz="0 0 0" rpy="1.5708 0 0"/>
-      <geometry>
-        <cylinder radius="0.03" length="0.02"/>
-      </geometry>
-    </collision>
-    <inertial>
-      <origin xyz="0 0 0" rpy="1.5708 0 0"/>
-      <mass value="0.2"/>
-      <inertia ixx="0.0001" ixy="0" ixz="0" iyy="0.0001" iyz="0" izz="0.0001"/>
+        <cylinder radius="0.06" length="0.04"/>
+      </geometry>
+      <material name="black"><color rgba="0 0 0 1"/></material>
+    </visual>
+    <collision>
+      <origin xyz="0 0 0" rpy="1.5708 0 0"/>
+      <geometry>
+        <cylinder radius="0.06" length="0.04"/>
+      </geometry>
+    </collision>
+    <inertial>
+      <mass value="0.8"/>
+      <inertia ixx="0.001" ixy="0" ixz="0" iyy="0.001" iyz="0" izz="0.001"/>
     </inertial>
   </link>
   <gazebo reference="wheel_fl">
-    <mu1>1.0</mu1>
-    <mu2>1.0</mu2>
-    <kp>1000000.0</kp>
-    <kd>100.0</kd>
+    <mu1>1000.0</mu1>
+    <mu2>1000.0</mu2>
     <material>Gazebo/Black</material>
   </gazebo>
-  <!-- Front Right Wheel -->
+  <joint name="wheel_fl_joint" type="continuous">
+    <parent link="base_link"/>
+    <child link="wheel_fl"/>
+    <origin xyz="0.12 0.11 0" rpy="0 0 0"/>
+    <axis xyz="0 1 0"/>
+  </joint>
   <link name="wheel_fr">
     <visual>
       <origin xyz="0 0 0" rpy="1.5708 0 0"/>
       <geometry>
-        <cylinder radius="0.03" length="0.02"/>
-      </geometry>
-      <material name="black">
-        <color rgba="0 0 0 1"/>
-      </material>
-    </visual>
-    <collision>
-      <origin xyz="0 0 0" rpy="1.5708 0 0"/>
-      <geometry>
-        <cylinder radius="0.03" length="0.02"/>
-      </geometry>
-    </collision>
-    <inertial>
-      <origin xyz="0 0 0" rpy="1.5708 0 0"/>
-      <mass value="0.2"/>
-      <inertia ixx="0.0001" ixy="0" ixz="0" iyy="0.0001" iyz="0" izz="0.0001"/>
+        <cylinder radius="0.06" length="0.04"/>
+      </geometry>
+      <material name="black"><color rgba="0 0 0 1"/></material>
+    </visual>
+    <collision>
+      <origin xyz="0 0 0" rpy="1.5708 0 0"/>
+      <geometry>
+        <cylinder radius="0.06" length="0.04"/>
+      </geometry>
+    </collision>
+    <inertial>
+      <mass value="0.8"/>
+      <inertia ixx="0.001" ixy="0" ixz="0" iyy="0.001" iyz="0" izz="0.001"/>
     </inertial>
   </link>
   <gazebo reference="wheel_fr">
-    <mu1>1.0</mu1>
-    <mu2>1.0</mu2>
-    <kp>1000000.0</kp>
-    <kd>100.0</kd>
+    <mu1>1000.0</mu1>
+    <mu2>1000.0</mu2>
     <material>Gazebo/Black</material>
   </gazebo>
-  <!-- Rear Left Wheel -->
+  <joint name="wheel_fr_joint" type="continuous">
+    <parent link="base_link"/>
+    <child link="wheel_fr"/>
+    <origin xyz="0.12 -0.11 0" rpy="0 0 0"/>
+    <axis xyz="0 1 0"/>
+  </joint>
   <link name="wheel_rl">
     <visual>
       <origin xyz="0 0 0" rpy="1.5708 0 0"/>
       <geometry>
-        <cylinder radius="0.03" length="0.02"/>
-      </geometry>
-      <material name="black">
-        <color rgba="0 0 0 1"/>
-      </material>
-    </visual>
-    <collision>
-      <origin xyz="0 0 0" rpy="1.5708 0 0"/>
-      <geometry>
-        <cylinder radius="0.03" length="0.02"/>
-      </geometry>
-    </collision>
-    <inertial>
-      <origin xyz="0 0 0" rpy="1.5708 0 0"/>
-      <mass value="0.2"/>
-      <inertia ixx="0.0001" ixy="0" ixz="0" iyy="0.0001" iyz="0" izz="0.0001"/>
+        <cylinder radius="0.06" length="0.04"/>
+      </geometry>
+      <material name="black"><color rgba="0 0 0 1"/></material>
+    </visual>
+    <collision>
+      <origin xyz="0 0 0" rpy="1.5708 0 0"/>
+      <geometry>
+        <cylinder radius="0.06" length="0.04"/>
+      </geometry>
+    </collision>
+    <inertial>
+      <mass value="0.8"/>
+      <inertia ixx="0.001" ixy="0" ixz="0" iyy="0.001" iyz="0" izz="0.001"/>
     </inertial>
   </link>
   <gazebo reference="wheel_rl">
-    <mu1>1.0</mu1>
-    <mu2>1.0</mu2>
-    <kp>1000000.0</kp>
-    <kd>100.0</kd>
+    <mu1>1000.0</mu1>
+    <mu2>1000.0</mu2>
     <material>Gazebo/Black</material>
   </gazebo>
-  <!-- Rear Right Wheel -->
+  <joint name="wheel_rl_joint" type="continuous">
+    <parent link="base_link"/>
+    <child link="wheel_rl"/>
+    <origin xyz="-0.12 0.11 0" rpy="0 0 0"/>
+    <axis xyz="0 1 0"/>
+  </joint>
   <link name="wheel_rr">
     <visual>
       <origin xyz="0 0 0" rpy="1.5708 0 0"/>
       <geometry>
-        <cylinder radius="0.03" length="0.02"/>
-      </geometry>
-      <material name="black">
-        <color rgba="0 0 0 1"/>
-      </material>
-    </visual>
-    <collision>
-      <origin xyz="0 0 0" rpy="1.5708 0 0"/>
-      <geometry>
-        <cylinder radius="0.03" length="0.02"/>
-      </geometry>
-    </collision>
-    <inertial>
-      <origin xyz="0 0 0" rpy="1.5708 0 0"/>
-      <mass value="0.2"/>
-      <inertia ixx="0.0001" ixy="0" ixz="0" iyy="0.0001" iyz="0" izz="0.0001"/>
+        <cylinder radius="0.06" length="0.04"/>
+      </geometry>
+      <material name="black"><color rgba="0 0 0 1"/></material>
+    </visual>
+    <collision>
+      <origin xyz="0 0 0" rpy="1.5708 0 0"/>
+      <geometry>
+        <cylinder radius="0.06" length="0.04"/>
+      </geometry>
+    </collision>
+    <inertial>
+      <mass value="0.8"/>
+      <inertia ixx="0.001" ixy="0" ixz="0" iyy="0.001" iyz="0" izz="0.001"/>
     </inertial>
   </link>
   <gazebo reference="wheel_rr">
-    <mu1>1.0</mu1>
-    <mu2>1.0</mu2>
-    <kp>1000000.0</kp>
-    <kd>100.0</kd>
+    <mu1>1000.0</mu1>
+    <mu2>1000.0</mu2>
     <material>Gazebo/Black</material>
   </gazebo>
-  <!-- Wheel joints -->
-  <joint name="joint_wheel_fl" type="continuous">
-    <parent link="base_link"/>
-    <child link="wheel_fl"/>
-    <origin xyz="0.12 0.09 -0.05" rpy="0 0 0"/>
+  <joint name="wheel_rr_joint" type="continuous">
+    <parent link="base_link"/>
+    <child link="wheel_rr"/>
+    <origin xyz="-0.12 -0.11 0" rpy="0 0 0"/>
     <axis xyz="0 1 0"/>
   </joint>
-  <joint name="joint_wheel_fr" type="continuous">
-    <parent link="base_link"/>
-    <child link="wheel_fr"/>
-    <origin xyz="0.12 -0.09 -0.05" rpy="0 0 0"/>
-    <axis xyz="0 1 0"/>
-  </joint>
-  <joint name="joint_wheel_rl" type="continuous">
-    <parent link="base_link"/>
-    <child link="wheel_rl"/>
-    <origin xyz="-0.12 0.09 -0.05" rpy="0 0 0"/>
-    <axis xyz="0 1 0"/>
-  </joint>
-  <joint name="joint_wheel_rr" type="continuous">
-    <parent link="base_link"/>
-    <child link="wheel_rr"/>
-    <origin xyz="-0.12 -0.09 -0.05" rpy="0 0 0"/>
-    <axis xyz="0 1 0"/>
-  </joint>
-  <!-- Front Ultrasonic Sensor Link -->
   <link name="ultrasonic_front">
     <visual>
-      <origin xyz="0 0 0" rpy="0 0 0"/>
-      <geometry>
-        <box size="0.02 0.04 0.015"/>
-      </geometry>
-      <material name="silver">
-        <color rgba="0.7 0.7 0.7 1"/>
-      </material>
-    </visual>
-    <collision>
-      <origin xyz="0 0 0" rpy="0 0 0"/>
-      <geometry>
-        <box size="0.02 0.04 0.015"/>
-      </geometry>
-    </collision>
-    <inertial>
-      <origin xyz="0 0 0" rpy="0 0 0"/>
+      <geometry>
+        <box size="0.02 0.03 0.01"/>
+      </geometry>
+      <material name="red"><color rgba="1 0 0 1"/></material>
+    </visual>
+    <inertial>
       <mass value="0.01"/>
-      <inertia ixx="0.00001" ixy="0" ixz="0" iyy="0.00001" iyz="0" izz="0.00001"/>
-    </inertial>
-  </link>
+      <inertia ixx="0.000001" ixy="0" ixz="0" iyy="0.000001" iyz="0" izz="0.000001"/>
+    </inertial>
+  </link>
+  <joint name="ultrasonic_front_joint" type="fixed">
+    <parent link="base_link"/>
+    <child link="ultrasonic_front"/>
+    <origin xyz="0.16 0 0.02" rpy="0 0 0"/>
+  </joint>
   <gazebo reference="ultrasonic_front">
-    <material>Gazebo/Grey</material>
-  </gazebo>
-  <!-- Front Ultrasonic Sensor Joint -->
-  <joint name="ultrasonic_front_joint" type="fixed">
-    <parent link="base_link"/>
-    <child link="ultrasonic_front"/>
-    <origin xyz="0.18 0 0.02" rpy="0 0 0"/>
-  </joint>
-  <!-- Front Ultrasonic Sensor Plugin -->
-  <gazebo reference="ultrasonic_front">
+    <material>Gazebo/Red</material>
     <sensor type="ray" name="ultrasonic_front_sensor">
-      <pose>0 0 0 0 0 0</pose>
       <visualize>true</visualize>
       <update_rate>10</update_rate>
@@ -214,28 +174,15 @@
         <scan>
           <horizontal>
-            <samples>5</samples>
-            <resolution>1</resolution>
-            <min_angle>-0.12</min_angle>
-            <max_angle>0.12</max_angle>
+            <samples>3</samples>
+            <min_angle>-0.1</min_angle>
+            <max_angle>0.1</max_angle>
           </horizontal>
-          <vertical>
-            <samples>5</samples>
-            <resolution>1</resolution>
-            <min_angle>-0.12</min_angle>
-            <max_angle>0.12</max_angle>
-          </vertical>
         </scan>
         <range>
-          <min>0.02</min>
+          <min>0.05</min>
           <max>4.0</max>
-          <resolution>0.01</resolution>
         </range>
-        <noise>
-          <type>gaussian</type>
-          <mean>0.0</mean>
-          <stddev>0.01</stddev>
-        </noise>
       </ray>
-      <plugin name="gazebo_ros_ultrasonic_front" filename="libgazebo_ros_ray_sensor.so">
+      <plugin name="ultrasonic_front_plugin" filename="libgazebo_ros_ray_sensor.so">
         <ros>
           <namespace>/pipe_bot</namespace>
@@ -243,44 +190,29 @@
         </ros>
         <output_type>sensor_msgs/Range</output_type>
+        <radiation_type>ultrasound</radiation_type>
         <frame_name>ultrasonic_front</frame_name>
       </plugin>
     </sensor>
   </gazebo>
-  <!-- Left Ultrasonic Sensor Link -->
   <link name="ultrasonic_left">
     <visual>
-      <origin xyz="0 0 0" rpy="0 0 0"/>
-      <geometry>
-        <box size="0.04 0.02 0.015"/>
-      </geometry>
-      <material name="silver">
-        <color rgba="0.7 0.7 0.7 1"/>
-      </material>
-    </visual>
-    <collision>
-      <origin xyz="0 0 0" rpy="0 0 0"/>
-      <geometry>
-        <box size="0.04 0.02 0.015"/>
-      </geometry>
-    </collision>
-    <inertial>
-      <origin xyz="0 0 0" rpy="0 0 0"/>
+      <geometry>
+        <box size="0.03 0.02 0.01"/>
+      </geometry>
+      <material name="red"><color rgba="1 0 0 1"/></material>
+    </visual>
+    <inertial>
       <mass value="0.01"/>
-      <inertia ixx="0.00001" ixy="0" ixz="0" iyy="0.00001" iyz="0" izz="0.00001"/>
-    </inertial>
-  </link>
+      <inertia ixx="0.000001" ixy="0" ixz="0" iyy="0.000001" iyz="0" izz="0.000001"/>
+    </inertial>
+  </link>
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